Commit message: change color of bot

File: GoChaseIt/catkin_ws/src/my_robot/urdf/my_robot.xacro (robot description, xacro)
@@ -2,4 +2,13 @@
 <robot name="my_robot" xmlns:xacro="http://www.ros.org/wiki/xacro">
     <xacro:include filename="$(find my_robot)/urdf/my_robot.gazebo" />
+    <gazebo reference="chassis">
+        <material>Gazebo/FlatBlack</material>
+    </gazebo>
+    <gazebo reference="left_wheel">
+        <material>Gazebo/Red</material>
+    </gazebo>
+    <gazebo reference="right_wheel">
+        <material>Gazebo/Red</material>
+    </gazebo>
     <link name="robot_footprint"></link>
     <joint name="robot_footprint_joint" type="fixed">
@@ -46,5 +55,6 @@
             <origin xyz="0 0 0" rpy=" 0 0 0" />
             <geometry>
-                <box size=".4 .2 .1" />
+                <box size=".4 .2 .1" color="red"/>
+                <color name="yellow"/>
             </geometry>
         </collision>

Commit message: adjust size

File: GoChaseIt/catkin_ws/src/my_robot/urdf/my_robot.xacro (robot description, xacro)
@@ -55,5 +55,5 @@
             <origin xyz="0 0 0" rpy=" 0 0 0" />
             <geometry>
-                <box size=".4 .2 .1" color="red"/>
+                <box size=".5 .2 .1" color="red"/>
                 <color name="yellow"/>
             </geometry>
@@ -62,5 +62,5 @@
             <origin xyz="0 0 0" rpy=" 0 0 0" />
             <geometry>
-                <box size=".4 .2 .1" />
+                <box size=".5 .2 .1" />
             </geometry>
         </visual>

Commit message: check if ball is too close

File: GoChaseIt/catkin_ws/src/my_robot/urdf/my_robot.xacro (robot description, xacro)
@@ -34,5 +34,5 @@
     </joint>
     <joint name="camera_joint" type="fixed">
-        <origin xyz="0.2 0 0 " rpy="0 0 0 "/>
+        <origin xyz="0.3 0 0 " rpy="0 0 0 "/>
         <axis xyz="0 1 0" rpy="0 0 0"/>
         <parent link="chassis"/>
